File: Charger.sch (EAGLE design)
At the start: 11 parts, among them IC1 MAX1044

Commit message: Changes in schematic and board to v1.1
Parts:
- +18V: device gm-supply:+18V(T) -> mb_supply:+18V(T)
- +9V: device gm-supply:+9V(T) -> mb_supply:+9V(T)
- C1: device gm-caps-electro-pol:0801 -> mb_caps-electro:0801
- C2, C3, C4: device gm-caps-electro-pol:0501 -> mb_caps-electro:0501
- D1: device gm-diodes:1N400X.3 -> mb_diodes:1N400X.3
- D2, D3: device gm-diodes:1N5817 -> mb_diodes:1N5817
- GND: device gm-supply:GND(T) -> mb_supply:GND(T)
- IC1: device gm-ics:MAX1044 -> mb_ics:MAX1044
Connections:
- removed net N$1: C1.-, IC1.3
- net GND: now also C1.-, IC1.3
Changed lines of the file:
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@@
 </classes>
 <parts>
-<part name="D1" library="gm-diodes" deviceset="1N400X" device=".3" value="1N4001"/>
-<part name="D2" library="gm-diodes" deviceset="1N5817" device=""/>
-<part name="D3" library="gm-diodes" deviceset="1N5817" device=""/>
-<part name="IC1" library="gm-ics" deviceset="MAX1044" device=""/>
-<part name="C1" library="gm-caps-electro-pol" deviceset="080" device="1" value="100uF"/>
-<part name="C2" library="gm-caps-electro-pol" deviceset="050" device="1" value="10uF"/>
-<part name="C3" library="gm-caps-electro-pol" deviceset="050" device="1" value="10uF"/>
-<part name="C4" library="gm-caps-electro-pol" deviceset="050" device="1" value="10uF"/>
-<part name="+18V" library="gm-supply" deviceset="+18V(T)" device=""/>
-<part name="+9V" library="gm-supply" deviceset="+9V(T)" device=""/>
-<part name="GND" library="gm-supply" deviceset="GND(T)" device=""/>
+<part name="D1" library="mb_diodes" deviceset="1N400X" device=".3" value="1N4001"/>
+<part name="D2" library="mb_diodes" deviceset="1N5817" device="" value="1N5817"/>
+<part name="D3" library="mb_diodes" deviceset="1N5817" device=""/>
+<part name="IC1" library="mb_ics" deviceset="MAX1044" device=""/>
+<part name="C1" library="mb_caps-electro" deviceset="080" device="1" value="100uF"/>
+<part name="C2" library="mb_caps-electro" deviceset="050" device="1" value="10uF"/>
+<part name="C3" library="mb_caps-electro" deviceset="050" device="1" value="10uF"/>
+<part name="C4" library="mb_caps-electro" deviceset="050" device="1" value="10uF"/>
+<part name="+18V" library="mb_supply" deviceset="+18V(T)" device=""/>
+<part name="+9V" library="mb_supply" deviceset="+9V(T)" device=""/>
+<part name="GND" library="mb_supply" deviceset="GND(T)" device=""/>
 <part name="GND1" library="gm-supply" deviceset="GND" device=""/>
 </parts>
@@
 <wire x1="0" y1="45.72" x2="0" y2="35.56" width="0.1524" layer="91"/>
 <pinref part="GND1" gate="GND" pin="GND"/>
-</segment>
-</net>
-<net name="N$1" class="0">
-<segment>
 <pinref part="C1" gate="G$1" pin="-"/>
 <pinref part="IC1" gate="G$1" pin="3"/>
 <wire x1="10.16" y1="45.72" x2="20.32" y2="45.72" width="0.1524" layer="91"/>
+<wire x1="10.16" y1="45.72" x2="0" y2="45.72" width="0.1524" layer="91"/>
+<junction x="10.16" y="45.72"/>
+<junction x="0" y="45.72"/>
 </segment>
 </net>
